File: V-0.2/schaltplan/Prototyp-V-0.2.brd (EAGLE design)
At the start: 160 x 100 mm, 49 parts, among them IC1 MEGA8-AI, IC2 NE5532N, X1 BU-SMB-H, X2 PN61729-S

Commit message: changes in the prototyp
Parts:
- added C15: 1µF, rcl:C025-024X044
- added IC3: AD5144A, analog-devices:TSSOP20
- added R6: 10k, rcl:0207/10
- added U$4: NJM78L03UA, linear:SOT89
- JP2: device jumper:JP2 -> jumper:JP4Q
- U$3: value AD5144A -> NJM79L03UA; device analog-devices:TSSOP20 -> linear:SOT89
- moved U$3 102.2 mm to (37.1, 83.5), flipped to the bottom, turned to 180 degrees
- moved C4 65.4 mm to (56.5, 33.0), turned to 180 degrees
- moved LED2 52.2 mm to (4.13, 30.8), turned to 180 degrees
- moved C5 46.3 mm to (10.8, 25.4), turned to 270 degrees
- moved Q1 35.0 mm to (15.2, 26.0), turned to 270 degrees
- moved R1 32.2 mm to (34.0, 28.9)
- moved R3 30.9 mm to (14.9, 30.8), turned to 180 degrees
- moved SV1 26.7 mm to (25.7, 42.2), turned to 180 degrees
- moved C7 22.5 mm to (15.9, 33.7)
- moved IC1 21.4 mm to (26.4, 27.9), turned to 135 degrees
- moved JP1 15.8 mm to (32.1, 19.1), turned to 270 degrees
- moved C13 10.2 mm to (79.4, 30.5)
- moved C10 7.89 mm to (44.1, 24.1)
- moved JP2 3.82 mm to (74.0, 34.3)
- moved R4 3.81 mm to (24.1, 20.3)
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Connections:
- new net +3V3: IC3.10, IC3.13, IC3.16, U$4.1
- new net -3V3: IC3.12, IC3.15, IC3.9, U$3.3
- new net N$32: C15.1, JP2.3
- new net N$33: IC3.5, IC3.6
- new net N$34: IC3.14, R10.1
- new net N$35: IC3.11, R6.1
- net +12V: now also U$4.3
- net -12V: now also U$3.2, U$3.2@1
- net AGND: now also IC3.7, IC3.8; no longer U$3.8
- net DGND: now also U$3.1, U$4.2, U$4.2@1
- net N$21: now also JP2.4, JP2.6, JP2.8
- net N$24: now also JP2.5; no longer JP2.1
- net N$26: now also JP2.1; no longer JP2.3
- net N$27: now also IC3.3, IC3.4; no longer U$3.6, U$3.7
- net N$28: now also C15.2, JP2.7
- net N$30: now also R6.2
