File: V-0.2/schaltplan/Signalgenerator-xmega.brd (EAGLE design)
At the start: 160 x 100 mm, 78 parts, among them IC2 NE5532N, IC3 AD5144A, IC4 XMEGA16C4AUR, X1 BU-SMB-H, X2 PN61729-S

Commit message: remove old folder
Routing:
- added copper zone on layer 16, net N$14
Other:
- board size 160 x 100 mm -> 255 x 100 mm
Changed lines of the file:
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@@
 <setting verticaltext="up"/>
 </settings>
-<grid distance="12.5" unitdist="mil" unit="mil" style="lines" multiple="1" display="no" altdistance="0.025" altunitdist="inch" altunit="inch"/>
+<grid distance="12.5" unitdist="mil" unit="mil" style="lines" multiple="1" display="yes" altdistance="0.025" altunitdist="inch" altunit="inch"/>
 <layers>
 <layer number="1" name="Top" color="4" fill="1" visible="yes" active="yes"/>
@@
 <layer number="43" name="vRestrict" color="2" fill="10" visible="yes" active="yes"/>
 <layer number="44" name="Drills" color="7" fill="1" visible="no" active="yes"/>
-<layer number="45" name="Holes" color="7" fill="1" visible="no" active="yes"/>
+<layer number="45" name="Holes" color="7" fill="1" visible="yes" active="yes"/>
 <layer number="46" name="Milling" color="3" fill="1" visible="no" active="yes"/>
 <layer number="47" name="Measures" color="7" fill="1" visible="no" active="yes"/>
@@
 <wire x1="160" y1="100" x2="0" y2="100" width="0" layer="20"/>
 <wire x1="0" y1="100" x2="0" y2="0" width="0" layer="20"/>
+<wire x1="-25" y1="60" x2="-90" y2="60" width="0.254" layer="20"/>
+<wire x1="-95" y1="55" x2="-95" y2="20" width="0.254" layer="20"/>
+<wire x1="-90" y1="15" x2="-25" y2="15" width="0.254" layer="20"/>
+<wire x1="-20" y1="20" x2="-20" y2="55" width="0.254" layer="20"/>
+<wire x1="-25" y1="60" x2="-20" y2="55" width="0.254" layer="20" curve="90"/>
+<wire x1="-25" y1="15" x2="-20" y2="20" width="0.254" layer="20" curve="-90"/>
+<wire x1="-90" y1="15" x2="-95" y2="20" width="0.254" layer="20" curve="90"/>
+<wire x1="-90" y1="60" x2="-95" y2="55" width="0.254" layer="20" curve="-90"/>
+<hole x="-90" y="55" drill="2"/>
+<hole x="-90" y="20" drill="2"/>
+<hole x="-25" y="20" drill="2"/>
+<hole x="-25" y="55" drill="2"/>
+<dimension x1="-95" y1="55" x2="-20" y2="55" x3="-57.5" y3="70" textsize="1.778" layer="21"/>
+<dimension x1="-90" y1="60" x2="-90" y2="15" x3="-100" y3="37.5" textsize="1.778" layer="21"/>
 </plain>
 <attributes>
@@
 </class>
 </classes>
-<designrules name="default">
+<designrules name="default *">
 <description language="de">&lt;b&gt;EAGLE Design Rules&lt;/b&gt;
 &lt;p&gt;
@@
 <param name="mdViaViaSameLayer" value="8mil"/>
 <param name="mnLayersViaInSmd" value="2"/>
-<param name="mdCopperDimension" value="40mil"/>
+<param name="mdCopperDimension" value="6mil"/>
 <param name="mdDrill" value="8mil"/>
 <param name="mdSmdStop" value="0mil"/>
@@
 <contactref element="IC4" pad="18"/>
 <contactref element="LED1" pad="K"/>
-<wire x1="60.96" y1="69.85" x2="60.96" y2="72.39" width="0" layer="19" extent="1-1"/>
-<wire x1="35.6485" y1="85.4835" x2="60.96" y2="72.39" width="0" layer="19" extent="16-16"/>
-<wire x1="31.75" y1="85.09" x2="35.6485" y2="85.4835" width="0" layer="19" extent="16-16"/>
-<wire x1="31.75" y1="87.63" x2="31.75" y2="85.09" width="0" layer="19" extent="1-1"/>
-<wire x1="36.195" y1="92.888" x2="31.75" y2="87.63" width="0" layer="19" extent="16-16"/>
-<wire x1="36.195" y1="95.555" x2="36.195" y2="92.888" width="0" layer="19" extent="16-16"/>
-<wire x1="31.75" y1="95.25" x2="36.195" y2="95.555" width="0" layer="19" extent="16-16"/>
-<wire x1="13.97" y1="90.134" x2="31.75" y2="87.63" width="0" layer="19" extent="16-16"/>
-<wire x1="19.0625" y1="68.665" x2="31.75" y2="85.09" width="0" layer="19" extent="16-16"/>
-<wire x1="23.2625" y1="62.065" x2="19.0625" y2="68.665" width="0" layer="19" extent="16-16"/>
-<wire x1="15.8625" y1="57.065" x2="23.2625" y2="62.065" width="0" layer="19" extent="16-16"/>
-<wire x1="11.6625" y1="62.065" x2="15.8625" y2="57.065" width="0" layer="19" extent="16-16"/>
-<wire x1="3.81" y1="22.53" x2="15.8625" y2="57.065" width="0" layer="19" extent="16-16"/>
-<wire x1="6.52" y1="15.26" x2="3.81" y2="22.53" width="0" layer="19" extent="1-1"/>
-<wire x1="3.81" y1="10.49" x2="6.52" y2="15.26" width="0" layer="19" extent="1-1"/>
-<wire x1="6.35" y1="5.08" x2="3.81" y2="10.49" width="0" layer="19" extent="1-1"/>
-<wire x1="25.4" y1="3.81" x2="6.35" y2="5.08" width="0" layer="19" extent="1-1"/>
-<wire x1="25.908" y1="11.43" x2="25.4" y2="3.81" width="0" layer="19" extent="1-1"/>
-<wire x1="42.3545" y1="24.13" x2="25.908" y2="11.43" width="0" layer="19" extent="1-1"/>
-<wire x1="57.155" y1="25.41" x2="42.3545" y2="24.13" width="0" layer="19" extent="16-16"/>
-<wire x1="60.96" y1="30.48" x2="57.155" y2="25.41" width="0" layer="19" extent="16-16"/>
-<wire x1="55.245" y1="33.02" x2="60.96" y2="30.48" width="0" layer="19" extent="1-1"/>
-<wire x1="48.387" y1="8.89" x2="42.3545" y2="24.13" width="0" layer="19" extent="1-1"/>
 </signal>
 <signal name="AGND">
@@
 <contactref element="IC4" pad="23"/>
 </signal>
+<signal name="N$14">
+<polygon width="0.254" layer="16" isolate="0.2032">
+<vertex x="-95" y="60"/>
+<vertex x="-20" y="60"/>
+<vertex x="-20" y="15"/>
+<vertex x="-95" y="15"/>
+</polygon>
+</signal>
 </signals>
