File: ReleaseCandidate/V1.0/version1.brd (EAGLE design)
At the start: 66 x 45 mm, 85 parts, among them IC1 ADG1604S, IC2 LM317MBSTT3, IC3 AD8610MR, IC4 AD8610MR, IC5 337IMP, Q1 16MHz, T1 BC847, T2 BC847, T3 BC847, T4 BC847, X2 BU-SMA-H

Commit message: make circuit diagramm beautifull, more layout
Parts:
- moved R22 10.9 mm to (33.3, 14.8)
- moved T1 6.99 mm to (33.2, 5.08), turned to 270 degrees
- moved T2 6.08 mm to (33.3, 8.89)
- moved R23 4.55 mm to (29.7, 10.5), turned to 180 degrees
- moved T4 0.22 mm to (21.0, 4.92)
Changed lines of the file:
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@@
 <element name="R20" library="rcl" package="R0603" value="10k" x="-72.39" y="71.12"/>
 <element name="R21" library="rcl" package="R0603" value="10k" x="-77.47" y="71.12"/>
-<element name="R22" library="rcl" package="R0603" value="10k" x="32.22625" y="3.96875" rot="MR0"/>
-<element name="R23" library="rcl" package="R0603" value="10k" x="33.655" y="8.255" rot="MR0"/>
+<element name="R22" library="rcl" package="R0603" value="10k" x="33.3375" y="14.76375" rot="MR0"/>
+<element name="R23" library="rcl" package="R0603" value="10k" x="29.68625" y="10.4775" rot="MR180"/>
 <element name="R24" library="rcl" package="R0603" value="10k" x="-26.67" y="76.2"/>
 <element name="R25" library="rcl" package="R0603" value="10k" x="-31.75" y="76.2"/>
@@
 <element name="SJ1" library="jumper" package="SJ_2" value="" x="6.50875" y="25.55875" rot="MR0"/>
 <element name="SJ2" library="jumper" package="SJ" value="" x="25.0825" y="15.5575" rot="R135"/>
-<element name="T1" library="transistor" package="SOT23" value="BC847" x="38.57625" y="9.525" rot="MR0"/>
-<element name="T2" library="transistor" package="SOT23" value="BC847" x="36.67125" y="3.81" rot="MR0"/>
+<element name="T1" library="transistor" package="SOT23" value="BC847" x="33.17875" y="5.08" rot="MR270"/>
+<element name="T2" library="transistor" package="SOT23" value="BC847" x="33.3375" y="8.89" rot="MR0"/>
 <element name="T3" library="transistor" package="SOT23" value="BC847" x="14.2875" y="3.81" rot="MR90"/>
-<element name="T4" library="transistor" package="SOT23" value="BC847" x="21.11375" y="5.08" rot="MR0"/>
+<element name="T4" library="transistor" package="SOT23" value="BC847" x="20.955" y="4.92125" rot="MR0"/>
 <element name="U$1" library="analog-devices" package="MSOP10" value="AD9833-SMD" x="49.2125" y="50.4825" rot="R90"/>
 <element name="U$2" library="linear" package="SOT23-5" value="LT1615" x="5.08" y="31.4325" rot="MR180"/>
@@
 <wire x1="53.575" y1="50.58095" x2="54.875" y2="50.58095" width="0" layer="19" extent="1-1"/>
 <wire x1="25.85125" y1="40.48125" x2="53.575" y2="50.58095" width="0" layer="19" extent="1-1"/>
-<wire x1="32.805" y1="8.255" x2="25.85125" y2="40.48125" width="0" layer="19" extent="1-16"/>
-<wire x1="31.37625" y1="3.96875" x2="32.805" y2="8.255" width="0" layer="19" extent="16-16"/>
+<wire x1="32.4875" y1="14.76375" x2="25.85125" y2="40.48125" width="0" layer="19" extent="1-16"/>
+<wire x1="30.53625" y1="10.4775" x2="32.4875" y2="14.76375" width="0" layer="19" extent="16-16"/>
 <wire x1="-25.82" y1="76.2" x2="25.85125" y2="40.48125" width="0" layer="19" extent="1-1"/>
 <wire x1="-30.9" y1="76.2" x2="-25.82" y2="76.2" width="0" layer="19" extent="1-1"/>
@@
 <contactref element="T4" pad="3"/>
 <contactref element="T3" pad="2"/>
-<wire x1="13.1875" y1="4.76" x2="21.11375" y2="6.18" width="0" layer="19" extent="16-16"/>
+<wire x1="13.1875" y1="4.76" x2="20.955" y2="6.02125" width="0" layer="19" extent="16-16"/>
 <wire x1="12.498215625" y1="11.36684375" x2="13.1875" y2="4.76" width="0" layer="19" extent="1-16"/>
 <wire x1="-78.32" y1="71.12" x2="12.498215625" y2="11.36684375" width="0" layer="19" extent="1-1"/>
@@
 <contactref element="T1" pad="3"/>
 <contactref element="T2" pad="2"/>
-<wire x1="35.72125" y1="2.71" x2="38.57625" y2="10.625" width="0" layer="19" extent="16-16"/>
-<wire x1="13.0639" y1="10.801159375" x2="35.72125" y2="2.71" width="0" layer="19" extent="1-16"/>
+<wire x1="32.07875" y1="5.08" x2="32.3875" y2="7.79" width="0" layer="19" extent="16-16"/>
+<wire x1="13.0639" y1="10.801159375" x2="32.3875" y2="7.79" width="0" layer="19" extent="1-16"/>
 <wire x1="-73.24" y1="71.12" x2="13.0639" y2="10.801159375" width="0" layer="19" extent="1-1"/>
 </signal>
@@
 <contactref element="T2" pad="1"/>
 <contactref element="R22" pad="1"/>
-<wire x1="37.62125" y1="2.71" x2="39.52625" y2="8.425" width="0" layer="19" extent="16-16"/>
-<wire x1="33.07625" y1="3.96875" x2="37.62125" y2="2.71" width="0" layer="19" extent="16-16"/>
+<wire x1="34.2875" y1="7.79" x2="34.1875" y2="14.76375" width="0" layer="19" extent="16-16"/>
+<wire x1="34.27875" y1="6.03" x2="34.2875" y2="7.79" width="0" layer="19" extent="16-16"/>
 </signal>
 <signal name="N$47">
@@
 <contactref element="T4" pad="1"/>
 <contactref element="R23" pad="1"/>
-<wire x1="22.06375" y1="3.98" x2="34.505" y2="8.255" width="0" layer="19" extent="16-16"/>
-<wire x1="13.1875" y1="2.86" x2="22.06375" y2="3.98" width="0" layer="19" extent="16-16"/>
+<wire x1="21.905" y1="3.82125" x2="28.83625" y2="10.4775" width="0" layer="19" extent="16-16"/>
+<wire x1="13.1875" y1="2.86" x2="21.905" y2="3.82125" width="0" layer="19" extent="16-16"/>
 </signal>
 <signal name="N$48">
@@
 <contactref element="T4" pad="2"/>
 <contactref element="T3" pad="3"/>
-<wire x1="20.16375" y1="3.98" x2="54.875" y2="56.41655" width="0" layer="19" extent="1-16"/>
-<wire x1="15.3875" y1="3.81" x2="20.16375" y2="3.98" width="0" layer="19" extent="16-16"/>
+<wire x1="20.005" y1="3.82125" x2="54.875" y2="56.41655" width="0" layer="19" extent="1-16"/>
+<wire x1="15.3875" y1="3.81" x2="20.005" y2="3.82125" width="0" layer="19" extent="16-16"/>
 <wire x1="-27.52" y1="76.2" x2="15.3875" y2="3.81" width="0" layer="19" extent="1-16"/>
 </signal>
@@
 <contactref element="T1" pad="2"/>
 <contactref element="T2" pad="3"/>
-<wire x1="37.62625" y1="8.425" x2="54.225" y2="56.41655" width="0" layer="19" extent="1-16"/>
-<wire x1="36.67125" y1="4.91" x2="37.62625" y2="8.425" width="0" layer="19" extent="16-16"/>
+<wire x1="33.3375" y1="9.99" x2="54.225" y2="56.41655" width="0" layer="19" extent="1-16"/>
+<wire x1="34.27875" y1="4.13" x2="33.3375" y2="9.99" width="0" layer="19" extent="16-16"/>
 <wire x1="-32.6" y1="76.2" x2="54.225" y2="56.41655" width="0" layer="19" extent="1-1"/>
 </signal>

Commit message: finish layout
Parts:
- added C31, C32, C33, C34: 100n, rcl:C0603
- added LED1: (no value), led:CHIP-LED0603
- added PAD1, PAD2, PAD3, PAD4: (no value), wirepad:SMD1,27-2,54
- added R26: 150, rcl:R0603
- moved R19 124.9 mm to (46.4, 19.4), turned to 270 degrees
- moved C30 121.7 mm to (36.2, 16.4), flipped to the bottom, turned to 270 degrees
- moved C29 118.0 mm to (40.0, 19.8), flipped to the bottom, turned to 270 degrees
- moved R21 112.9 mm to (15.7, 7.30), flipped to the bottom, turned to 90 degrees
- moved R20 110.6 mm to (17.9, 7.30), flipped to the bottom, turned to 90 degrees
- moved R13 105.9 mm to (47.1, 22.5), turned to 180 degrees
- moved C10 104.6 mm to (22.1, 21.7), turned to 180 degrees
- moved R6 101.8 mm to (23.3, 13.8), flipped to the bottom
- moved R5 99.8 mm to (20.8, 7.94), turned to 90 degrees
- moved R12 98.5 mm to (43.2, 21.6), turned to 270 degrees
- moved R11 98.4 mm to (47.9, 26.2), turned to 90 degrees
- moved R14 93.8 mm to (47.0, 29.1), turned to 180 degrees
- moved C9 93.0 mm to (17.0, 24.6), turned to 225 degrees
- moved R4 92.9 mm to (23.3, 15.6), flipped to the bottom
- moved C3 91.7 mm to (7.46, 18.9), turned to 225 degrees
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Connections:
- new net N$50: PAD2.1, U$3.11
- new net N$51: LED1.A, R26.1
- net +12V: now also C31.2, C33.2
- net -12V: now also C32.1, C34.1
- net AGND: now also C31.1, C32.2, C33.1, C34.2, IC4.3, U$6.14, U$6.15
- net GND: now also LED1.C; no longer IC4.2, U$6.14, U$6.15
- net N$32: now also IC4.2; no longer IC4.3
- net N$4: now also PAD3.1
- net N$8: now also PAD1.1
- net N$9: now also PAD4.1
- net VCC: now also R26.2
Routing:
- net +3V3: track 0.00 -> 98.4 mm, vias 0 -> 5
- net VCC: track 14.2 -> 91.2 mm, vias 1 -> 4
- net +12V: track 2.13 -> 61.6 mm, vias 1 -> 3
- net -12V: track 2.72 -> 54.1 mm, vias 1 -> 2
- net -3V3: track 0.00 -> 47.2 mm, vias 0 -> 3
- net N$48: track 0.00 -> 38.1 mm, vias 0 -> 2
- net N$49: track 0.00 -> 36.6 mm, vias 0 -> 3
- net N$20: track 0.00 -> 33.9 mm, vias 0 -> 2
- net N$22: track 0.00 -> 24.6 mm, vias 0 -> 3
- net N$34: track 0.00 -> 23.7 mm, vias 0 -> 2
- net N$45: track 0.00 -> 20.4 mm, vias 0 -> 1
- net N$42: track 0.00 -> 19.9 mm, vias 0 -> 1
- net N$43: track 0.00 -> 18.9 mm, vias 0 -> 1
- net N$19: track 0.00 -> 16.4 mm, vias 0 -> 1
- net N$33: track 0.00 -> 14.7 mm, vias 0 -> 1
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Other:
- board text added: "(c)2015 Hendrik Lüth LabConnect Signalgenerator github.com/labconnect"
