File: ReleaseCandidate/V1.0/version1-biene.brd (EAGLE design)
At the start: 66 x 45 mm, 96 parts, among them IC1 ADG1604S, IC2 LM317MBSTT3, IC3 AD8610MR, IC4 AD8610MR, IC5 337IMP, Q1 16MHz, T1 BC847, T2 BC847, T3 BC847, T4 BC847, X2 BU-SMA-H

Commit message: crate gerber files for the pcb with the bee
Parts:
- moved U$12 2.29 mm to (32.1, 3.02)
Other:
- board text added: "Dirty White Signalgenerator"
