File: schematics/V1.0/version1-biene.brd (EAGLE design)
At the start: 66 x 45 mm, 96 parts, among them IC1 ADG1604S, IC2 LM317MBSTT3, IC3 AD8610MR, IC4 AD8610MR, IC5 337IMP, Q1 16MHz, T1 BC847, T2 BC847, T3 BC847, T4 BC847, X2 BU-SMA-H

Commit message: change values, more usb-protokoll
Parts:
- C1, C2: value 22n -> 22p
Changed lines of the file:
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@@
 </autorouter>
 <elements>
-<element name="C1" library="rcl" package="C0603" value="22n" x="4.7625" y="4.28625" rot="R90"/>
+<element name="C1" library="rcl" package="C0603" value="22p" x="4.7625" y="4.28625" rot="R90"/>
 <element name="C10" library="rcl" package="C0603" value="100n" x="22.06625" y="21.74875" rot="R180"/>
 <element name="C11" library="rcl" package="SMC_B" value="" x="28.2575" y="24.92375" rot="R90"/>
@@
 </element>
 <element name="C19" library="rcl" package="SMC_A" value="1µF" x="7.14375" y="30.95625" rot="R90"/>
-<element name="C2" library="rcl" package="C0603" value="22n" x="4.92125" y="12.54125"/>
+<element name="C2" library="rcl" package="C0603" value="22p" x="4.92125" y="12.54125"/>
 <element name="C20" library="rcl" package="C0603" value="100n" x="11.1125" y="24.765" rot="R180"/>
 <element name="C21" library="rcl" package="C0603" value="100n" x="14.44625" y="35.56" rot="R90"/>

Commit message: change circuit, add new picture
Routing:
- net N$53: track 3.29 -> 0.00 mm
Changed lines of the file:
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@@
 <wire x1="9.68375" y1="21.11375" x2="8.521909375" y2="19.951909375" width="0.254" layer="1"/>
-</signal>
-<signal name="N$53">
-<contactref element="U$3" pad="2"/>
-<contactref element="C20" pad="1"/>
-<wire x1="14.195271875" y1="22.397709375" x2="11.9625" y2="24.63048125" width="0.254" layer="1"/>
-<wire x1="11.9625" y1="24.63048125" x2="11.9625" y2="24.765" width="0.254" layer="1"/>
 </signal>
 <signal name="N$3">
@@
 <wire x1="8.21125" y1="25.1825" x2="8.21125" y2="26.67" width="0.254" layer="1"/>
 </signal>
+<signal name="N$53">
+<contactref element="C20" pad="1"/>
+<contactref element="U$3" pad="2"/>
+<wire x1="14.195271875" y1="22.397709375" x2="11.9625" y2="24.765" width="0" layer="19" extent="1-1"/>
+</signal>
 </signals>
