File: schematics/V1.0/version1-biene.sch (EAGLE design)
At the start: 95 parts, among them IC1 ADG1604S, IC2 LM317MBSTT3, IC3 AD8610MR, IC4 AD8610MR, IC5 337IMP, Q1 16MHz, T1 BC847, T2 BC847, T3 BC847, T4 BC847, X2 BU-SMA-H

Commit message: change values, more usb-protokoll
Parts:
- C1, C2: value 22n -> 22p
Changed lines of the file:
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@@
 </classes>
 <parts>
-<part name="C1" library="rcl" deviceset="C-EU" device="C0603" value="22n"/>
-<part name="C2" library="rcl" deviceset="C-EU" device="C0603" value="22n"/>
+<part name="C1" library="rcl" deviceset="C-EU" device="C0603" value="22p"/>
+<part name="C2" library="rcl" deviceset="C-EU" device="C0603" value="22p"/>
 <part name="GND1" library="supply1" deviceset="GND" device=""/>
 <part name="P+1" library="supply1" deviceset="VCC" device=""/>
