File: schematics/V1.0/version1.brd (EAGLE design)
At the start: 66 x 45 mm, 95 parts, among them IC1 ADG1604S, IC2 LM317MBSTT3, IC3 AD8610MR, IC4 AD8610MR, IC5 337IMP, Q1 16MHz, T1 BC847, T2 BC847, T3 BC847, T4 BC847, X2 BU-SMA-H

Commit message: change circuit, add new picture
Connections:
- removed net N$53: C20.1, U$3.2
- net VCC: now also C20.1, U$3.2
Routing:
- net VCC: track 91.2 -> 97.8 mm, vias 4 -> 6
- net N$53: track 3.29 -> 0.00 mm
Changed lines of the file:
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@@
 <layers>
 <layer number="1" name="Top" color="4" fill="1" visible="yes" active="yes"/>
-<layer number="16" name="Bottom" color="1" fill="1" visible="no" active="yes"/>
+<layer number="16" name="Bottom" color="1" fill="1" visible="yes" active="yes"/>
 <layer number="17" name="Pads" color="2" fill="1" visible="yes" active="yes"/>
 <layer number="18" name="Vias" color="2" fill="1" visible="yes" active="yes"/>
@@
 <layer number="20" name="Dimension" color="15" fill="1" visible="yes" active="yes"/>
 <layer number="21" name="tPlace" color="7" fill="1" visible="yes" active="yes"/>
-<layer number="22" name="bPlace" color="7" fill="1" visible="no" active="yes"/>
+<layer number="22" name="bPlace" color="7" fill="1" visible="yes" active="yes"/>
 <layer number="23" name="tOrigins" color="15" fill="1" visible="yes" active="yes"/>
-<layer number="24" name="bOrigins" color="15" fill="1" visible="no" active="yes"/>
+<layer number="24" name="bOrigins" color="15" fill="1" visible="yes" active="yes"/>
 <layer number="25" name="tNames" color="7" fill="1" visible="yes" active="yes"/>
-<layer number="26" name="bNames" color="7" fill="1" visible="no" active="yes"/>
+<layer number="26" name="bNames" color="7" fill="1" visible="yes" active="yes"/>
 <layer number="27" name="tValues" color="7" fill="1" visible="yes" active="yes"/>
-<layer number="28" name="bValues" color="7" fill="1" visible="no" active="yes"/>
+<layer number="28" name="bValues" color="7" fill="1" visible="yes" active="yes"/>
 <layer number="29" name="tStop" color="7" fill="3" visible="no" active="yes"/>
 <layer number="30" name="bStop" color="7" fill="6" visible="no" active="yes"/>
@@
 <wire x1="6.61125" y1="25.0825" x2="6.4525" y2="24.92375" width="0.254" layer="1"/>
 <wire x1="6.4525" y1="24.92375" x2="4.1275" y2="24.92375" width="0.254" layer="1"/>
+<contactref element="C20" pad="1"/>
+<contactref element="U$3" pad="2"/>
+<wire x1="11.9625" y1="24.63048125" x2="11.9625" y2="24.765" width="0.254" layer="1"/>
+<wire x1="14.195271875" y1="22.397709375" x2="13.335" y2="23.25798125" width="0.254" layer="1"/>
+<wire x1="13.335" y1="23.25798125" x2="13.335" y2="23.33625" width="0.254" layer="1"/>
+<via x="13.335" y="23.33625" extent="1-16" drill="0.3048" shape="octagon"/>
+<wire x1="13.335" y1="23.33625" x2="13.49375" y2="23.495" width="0.254" layer="16"/>
+<wire x1="13.49375" y1="23.495" x2="15.875" y2="23.495" width="0.254" layer="16"/>
+<wire x1="15.875" y1="23.495" x2="16.35125" y2="23.97125" width="0.254" layer="16"/>
+<via x="16.35125" y="23.97125" extent="1-16" drill="0.3048" shape="octagon"/>
+<wire x1="16.35125" y1="23.97125" x2="16.38520625" y2="24.00520625" width="0.254" layer="1"/>
+<wire x1="11.9625" y1="24.63048125" x2="13.25673125" y2="23.33625" width="0.254" layer="1"/>
+<wire x1="13.25673125" y1="23.33625" x2="13.335" y2="23.33625" width="0.254" layer="1"/>
 </signal>
 <signal name="N$8">
@@
 <wire x1="9.68375" y1="21.11375" x2="8.521909375" y2="19.951909375" width="0.254" layer="1"/>
 </signal>
-<signal name="N$53">
-<contactref element="U$3" pad="2"/>
-<contactref element="C20" pad="1"/>
-<wire x1="14.195271875" y1="22.397709375" x2="11.9625" y2="24.63048125" width="0.254" layer="1"/>
-<wire x1="11.9625" y1="24.63048125" x2="11.9625" y2="24.765" width="0.254" layer="1"/>
-</signal>
 <signal name="N$3">
