File: schematics/V1.0/version1.sch (EAGLE design)
At the start: 94 parts, among them IC1 ADG1604S, IC2 LM317MBSTT3, IC3 AD8610MR, IC4 AD8610MR, IC5 337IMP, Q1 16MHz, T1 BC847, T2 BC847, T3 BC847, T4 BC847, X2 BU-SMA-H

Commit message: change circuit, add new picture
Connections:
- removed net N$53: C20.1, U$3.UVCC
- net VCC: now also C20.1, U$3.UVCC
Changed lines of the file:
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@@
 <junction x="27.94" y="93.98"/>
 <pinref part="U$3" gate="G$1" pin="VBUS"/>
-<wire x1="38.1" y1="83.82" x2="27.94" y2="83.82" width="0.1524" layer="91"/>
+<wire x1="38.1" y1="83.82" x2="30.48" y2="83.82" width="0.1524" layer="91"/>
+<wire x1="30.48" y1="83.82" x2="27.94" y2="83.82" width="0.1524" layer="91"/>
 <wire x1="27.94" y1="83.82" x2="27.94" y2="91.44" width="0.1524" layer="91"/>
 <junction x="27.94" y="91.44"/>
+<pinref part="U$3" gate="G$1" pin="UVCC"/>
+<pinref part="C20" gate="G$1" pin="1"/>
+<wire x1="38.1" y1="81.28" x2="30.48" y2="81.28" width="0.1524" layer="91"/>
+<wire x1="30.48" y1="81.28" x2="27.94" y2="81.28" width="0.1524" layer="91"/>
+<wire x1="30.48" y1="81.28" x2="30.48" y2="83.82" width="0.1524" layer="91"/>
+<junction x="30.48" y="81.28"/>
+<junction x="30.48" y="83.82"/>
 </segment>
 <segment>
@@
 </segment>
 </net>
-<net name="N$53" class="0">
-<segment>
-<pinref part="U$3" gate="G$1" pin="UVCC"/>
-<pinref part="C20" gate="G$1" pin="1"/>
-<wire x1="38.1" y1="81.28" x2="27.94" y2="81.28" width="0.1524" layer="91"/>
-</segment>
-</net>
